Commit message: modified urdf

File: arm_description/urdf/arm_description.urdf (robot description, URDF)
Before this commit: robot arm_description, 7 links, 6 joints
Joints:
- joint actuator_joint: limit lower=-0.6 upper=+0.6 effort=100 velocity=50 -> lower=-1.0 upper=+1.0 effort=100 velocity=50
- joint differential_joint: limit lower=-0.6 upper=+0.6 effort=100 velocity=50 -> lower=-1.0 upper=+1.0 effort=100 velocity=50
- joint differential_rotation_joint: limit lower=-0.6 upper=+0.6 effort=100 velocity=50 -> lower=-1.0 upper=+1.0 effort=100 velocity=50
- joint elbow_joint: limit lower=-0.6 upper=+0.6 effort=100 velocity=50 -> lower=-1.0 upper=+1.0 effort=100 velocity=50
- joint shoulder_joint: limit lower=-0.6 upper=+0.6 effort=100 velocity=50 -> lower=-1.0 upper=+1.0 effort=100 velocity=50
